File: PVC Junction Box Modules/CONTROL circuit for Junction Box v2.sch (EAGLE design)
At the start: 44 parts, among them IC5 1117-33, Q24 A03400

Commit message: save
Other:
- note removed: "USB TO SERIAL"
Changed lines of the file:
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@@
 <wire x1="359.41" y1="-156.21" x2="359.41" y2="-53.34" width="0.1524" layer="95"/>
 <wire x1="359.41" y1="-53.34" x2="218.44" y2="-53.34" width="0.1524" layer="95"/>
-<text x="218.44" y="-52.07" size="3.81" layer="95">USB TO SERIAL</text>
 <text x="386.08" y="-121.92" size="6.4516" layer="91">TODO
 ir recv
