File: ESP32 Alarm/ESP32 Alarm.brd (EAGLE design)
At the start: 100 x 95 mm, 127 parts, among them IC1 TLC339P, IC2 TLC339P, IC3 TLC339P, IC4 TLC339P, IC5 XL1509, IC6 1117-33, J1 JRC-21F-4100, Q1 200mA/40V, Q10 60V/32A/35mΩ, Q11 200mA/40V, Q2 200mA/40V, Q3 60V/32A/35mΩ, Q4 60V/32A/35mΩ, Q5 60V/32A/35mΩ, Q6 60V/32A/35mΩ, Q7 60V/32A/35mΩ, Q8 60V/32A/35mΩ, Q9 60V/32A/35mΩ, X10 MCV2, X11 MCV2, X12 MCV2, X13 MCV2, X14 MCV2, X15 MCV2, X16 MCV2, X17 MCV2, X18 MCV2, X19 MCV3, X3 MCV2, X4 MCV2, X5 MCV2, X6 MCV2, X7 MCV2, X8 MCV2, X9 MCV2

Commit message: update
Parts:
- removed J3: (no value), SparkFun-Connectors:1X04_LOCK
- Q3: value 60V/32A/35mΩ -> 35A/25V/8.5mΩ; device SparkFun-DiscreteSemi:TO220V -> SparkFun-DiscreteSemi:DPAK
Connections:
- net 3.3V: no longer J3.2
- net GND: no longer J3.1
- net GPIO4: no longer J3.3
- net GPIO5: no longer J3.4
- net N$41: now also Q3.4; no longer Q3.2
Routing:
- net N$37: track 11.2 -> 16.6 mm
- net GPIO5: track 36.4 -> 33.2 mm
- net GPIO4: track 41.6 -> 38.6 mm
- net 3.3V: track 242.9 -> 241.3 mm
