File: ESP32 Alarm/ESP32 Alarm.sch (EAGLE design)
At the start: 127 parts, among them IC1 TLC339P, IC2 TLC339P, IC3 TLC339P, IC4 TLC339P, IC5 XL1509, IC6 1117-33, J1 JRC-21F-4100, Q1 200mA/40V, Q10 60V/32A/35mΩ, Q11 200mA/40V, Q2 200mA/40V, Q3 60V/32A/35mΩ, Q4 60V/32A/35mΩ, Q5 60V/32A/35mΩ, Q6 60V/32A/35mΩ, Q7 60V/32A/35mΩ, Q8 60V/32A/35mΩ, Q9 60V/32A/35mΩ, X10 MCV2, X11 MCV2, X12 MCV2, X13 MCV2, X14 MCV2, X15 MCV2, X16 MCV2, X17 MCV2, X18 MCV2, X19 MCV3, X3 MCV2, X4 MCV2, X5 MCV2, X6 MCV2, X7 MCV2, X8 MCV2, X9 MCV2

Commit message: update
Parts:
- removed J3: (no value), SparkFun-Connectors:CONN_04LOCK
- Q3: value 60V/32A/35mΩ -> 35A/25V/8.5mΩ; device SparkFun-DiscreteSemi:MOSFET-NCH-FQP30N06L -> SparkFun-DiscreteSemi:MOSFET-NCH-FDD8780
Connections:
- net 3.3V: no longer J3.2
- net GND: no longer J3.1
- net GPIO4: no longer J3.3
- net GPIO5: no longer J3.4
Changed lines of the file:
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@@
 <part name="X17" library="con-phoenix-381_l" deviceset="MCV2" device=""/>
 <part name="X18" library="con-phoenix-381_l" deviceset="MCV2" device=""/>
-<part name="Q3" library="SparkFun-DiscreteSemi" library_urn="urn:adsk.eagle:library:514" deviceset="MOSFET-NCH" device="-FQP30N06L" package3d_urn="urn:adsk.eagle:package:38447/1" value="60V/32A/35mΩ"/>
+<part name="Q3" library="SparkFun-DiscreteSemi" library_urn="urn:adsk.eagle:library:514" deviceset="MOSFET-NCH" device="-FDD8780" package3d_urn="urn:adsk.eagle:package:38459/1" value="35A/25V/8.5mΩ"/>
 <part name="Q4" library="SparkFun-DiscreteSemi" library_urn="urn:adsk.eagle:library:514" deviceset="MOSFET-NCH" device="-FQP30N06L" package3d_urn="urn:adsk.eagle:package:38447/1" value="60V/32A/35mΩ"/>
 <part name="Q5" library="SparkFun-DiscreteSemi" library_urn="urn:adsk.eagle:library:514" deviceset="MOSFET-NCH" device="-FQP30N06L" package3d_urn="urn:adsk.eagle:package:38447/1" value="60V/32A/35mΩ"/>
@@
 <part name="J2" library="SparkFun-Connectors" library_urn="urn:adsk.eagle:library:513" deviceset="CONN_04" device="LOCK" package3d_urn="urn:adsk.eagle:package:38089/1"/>
 <part name="C1" library="SparkFun" deviceset="CAP_POL" device="1206" value="10uF"/>
-<part name="J3" library="SparkFun-Connectors" library_urn="urn:adsk.eagle:library:513" deviceset="CONN_04" device="LOCK" package3d_urn="urn:adsk.eagle:package:38089/1"/>
 <part name="IC6" library="v-reg" library_urn="urn:adsk.eagle:library:409" deviceset="LD117A?*" device="S" package3d_urn="urn:adsk.eagle:package:30370/1" technology="33TR" value="1117-33"/>
 <part name="C7" library="SparkFun" deviceset="CAP_POL" device="1206" value="10uF"/>
@@
 <attribute name="VALUE" x="477.266" y="-108.331" size="1.778" layer="96"/>
 </instance>
-<instance part="J3" gate="G$1" x="450.85" y="-125.73" smashed="yes">
-<attribute name="VALUE" x="445.77" y="-133.096" size="1.778" layer="96" font="vector"/>
-<attribute name="NAME" x="445.77" y="-117.602" size="1.778" layer="95" font="vector"/>
-</instance>
 <instance part="IC6" gate="G$1" x="345.186" y="22.987" smashed="yes">
 <attribute name="NAME" x="347.726" y="15.367" size="1.778" layer="95"/>
@@
 <label x="461.01" y="-101.6" size="1.778" layer="95"/>
 <pinref part="C1" gate="G$1" pin="+"/>
-<wire x1="455.93" y1="-101.6" x2="473.71" y2="-101.6" width="0.1524" layer="91"/>
-<pinref part="J3" gate="G$1" pin="2"/>
-<wire x1="473.71" y1="-101.6" x2="476.25" y2="-101.6" width="0.1524" layer="91"/>
-<wire x1="455.93" y1="-125.73" x2="473.71" y2="-125.73" width="0.1524" layer="91"/>
-<wire x1="473.71" y1="-125.73" x2="473.71" y2="-101.6" width="0.1524" layer="91"/>
-<junction x="473.71" y="-101.6"/>
+<wire x1="455.93" y1="-101.6" x2="476.25" y2="-101.6" width="0.1524" layer="91"/>
 </segment>
 <segment>
@@
 <pinref part="C1" gate="G$1" pin="-"/>
 <wire x1="455.93" y1="-109.22" x2="476.25" y2="-109.22" width="0.1524" layer="91"/>
-<pinref part="J3" gate="G$1" pin="1"/>
-<wire x1="455.93" y1="-128.27" x2="476.25" y2="-128.27" width="0.1524" layer="91"/>
-<wire x1="476.25" y1="-128.27" x2="476.25" y2="-109.22" width="0.1524" layer="91"/>
-<junction x="476.25" y="-109.22"/>
 </segment>
 <segment>
@@
 <label x="137.16" y="-17.78" size="1.778" layer="95"/>
 </segment>
-<segment>
-<pinref part="J3" gate="G$1" pin="3"/>
-<wire x1="455.93" y1="-123.19" x2="469.9" y2="-123.19" width="0.1524" layer="91"/>
-<label x="462.28" y="-123.19" size="1.778" layer="95"/>
-</segment>
 </net>
 <net name="N$57" class="0">
@@
 <label x="137.16" y="-20.32" size="1.778" layer="95"/>
 </segment>
-<segment>
-<pinref part="J3" gate="G$1" pin="4"/>
-<wire x1="455.93" y1="-120.65" x2="469.9" y2="-120.65" width="0.1524" layer="91"/>
-<label x="462.28" y="-120.65" size="1.778" layer="95"/>
-</segment>
-</net>
+</net>
