File: Solar ESP Modules/Solar Power Management ESP32.brd (EAGLE design)
At the start: 90 x 80 mm, 35 parts, among them IC1 TP4056, IC5 1117-33, Q1 FDN360P, U2 ESP-WROOM-32NARROW

Commit message: save
Parts:
- removed D1: MBRA210LT3, microbuilder:SMADIODE
- removed R11, R12, R13, R14, R8: 1K, rcl:R1206
- added BZ1, BZ2, SZ1, SZ2: (no value), rcl:R1206
- added C14, C16: 0.1uF, SparkFun:0603-CAP
- added C15, C4, C5: 10uF, SparkFun:EIA3216
- added D21: RED/GRN BICOLOR 3528 LED, Wurth_Elektronik_Optoelectronics_rev15c:3528
- added IC2: 1117-33, v-reg:SOT223
- added J1, J2: (no value), SparkFun-Connectors2:2X3-SHROUDED
- added J3: USB-C-Socket, SparkFun-Connectors:USB-C-16P
- added R1, R21: 10k, SparkFun-Resistors:0603
- added R22, R27: 5.1k, SparkFun-Resistors:0603@1
- added R30, R31: 1K, SparkFun:0603-RES
- added SJ1, SJ2: (no value), jumper:SJ
- added T3, T4: MBT2N2222, transistor:SOT23-BEC
- added U6: FT232RLSSOP, SparkFun:SSOP28DB
- C1: device rcl:C1206@1 -> rcl:C1206
- moved IO0 79.5 mm to (5.00, 37.0), turned to 180 degrees
- moved RESET 79.5 mm to (5.00, 52.0), turned to 180 degrees
- moved R10 30.0 mm to (26.1, 39.9)
- moved C6 29.9 mm to (26.1, 45.9)
- moved U2 25.0 mm to (45.0, 40.5)
- moved C3 19.7 mm to (26.1, 42.9), turned to 180 degrees
- moved IC5 18.6 mm to (16.5, 50.5), turned to 0 degrees
- moved C13 15.5 mm to (26.1, 49.9), turned to 180 degrees
- moved C12 12.5 mm to (17.0, 43.5), turned to 0 degrees
- moved D11 12.1 mm to (16.5, 39.4), turned to 0 degrees
- moved R15 2.70 mm to (27.3, 85.1)
- moved SOLAR-IN 1.00 mm to (18.0, 24.5)
- moved BATT+ 0.50 mm to (81.4, 69.2)
- moved BATT- 0.50 mm to (8.90, 69.2)
- moved Q1 0.32 mm to (34.9, 84.7)
Connections:
- removed net N$2: Q1.1, R15.2, R8.2
- new net 26_BEEPER: U2.11
- new net 3VUSB: C16.1, U6.17, U6.4
- new net CC1: J3.A5, R27.2
- new net CC2: J3.B5, R22.2
- new net CTS: U6.11
- new net D+1: J3.A6, J3.B6, U6.15
- new net D-1: J3.A7, J3.B7, U6.16
- new net DTR: R1.1, T3.E, U6.2
- new net N$4: R1.2, T4.B
- new net N$6: R21.2, T3.B
- new net N$7: D21.4, R30.2
- new net N$9: D21.3, R31.2
- new net RTS: R21.1, T4.E, U6.3
- new net RXLED: R30.1, U6.22
- new net SHLD: J3.SHLD1, J3.SHLD2, J3.SHLD3, J3.SHLD4, J3.SHLD5, J3.SHLD6, J3.SHLD7, J3.SHLD8
- new net TXLED: R31.1, U6.23
- net 0: now also J1.6, J2.6, T3.C
- net 3.3V: now also C5.A, IC2.4, J1.2, J2.2
- net BATT+: now also BZ1.1; no longer R11.1
- net BATT-VOLTAGE-ADC: now also BZ1.2, BZ2.1, SJ2.1, SJ2.2, U2.5; no longer R11.2, R12.1, U2.7
- net CHIP_PU: now also J1.1, J2.1, T4.C
- net GND: now also BZ2.2, C14.2, C15.C, C16.2, C4.C, C5.C, IC2.1, J1.4, J2.4, J3.GND, J3.GND2, R22.1, R27.1, SZ2.2, U6.18, U6.21, U6.25, U6.26, U6.7; no longer R12.2, R14.2
- net RX: now also J1.3, J2.3, U6.5
- net SOLAR+: now also Q1.1, R15.2, SZ1.1; no longer R13.1
- net SOLAR-VOLTAGE-ADC: now also SJ1.1, SJ1.2, SZ1.2, SZ2.1, U2.4; no longer R13.2, R14.1, U2.6
- net TX: now also J1.5, J2.5, U6.1
- net VBUS: now also C14.1, C15.A, C4.A, D21.1, D21.2, IC2.3, J3.VBUS1, J3.VBUS2, U6.20; no longer D1.A, R8.1
- net VCC: no longer D1.C
Routing:
- net SOLAR+: track 28.1 -> 173.0 mm, vias 0 -> 2
- net VCC: track 0.00 -> 98.3 mm
- net CHIP_PU: track 4.50 -> 91.3 mm, vias 0 -> 3
- net BATT+: track 0.00 -> 86.1 mm
- net 0: track 0.00 -> 81.0 mm, vias 0 -> 2
- net 3.3V: track 9.09 -> 74.6 mm, vias 0 -> 1
- net VBUS: track 0.00 -> 62.8 mm, vias 0 -> 2
- net RX: track 0.00 -> 57.0 mm, vias 0 -> 1
- net TX: track 0.00 -> 49.4 mm, vias 0 -> 1
- net DTR: track 0.00 -> 25.8 mm
- net GND: track 16.4 -> 38.3 mm, vias 4 -> 17
- net 3VUSB: track 0.00 -> 14.6 mm
- net RTS: track 0.00 -> 14.2 mm
- net SOLAR-VOLTAGE-ADC: track 7.51 -> 19.6 mm
- net D-1: track 0.00 -> 11.1 mm
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Other:
- board size 90 x 80 mm -> 90 x 90 mm
- board text added: "3V3"
- board text added: "5V-8V"
- board text added: "ESProg"
- board text added: "GND"
- board text added: "IO0"
- board text added: "RST"
- board text added: "RX"
- board text added: "TX"

Commit message: update
Parts:
- added U$3: XKBENTERPRISESS-12D11G5R, XKB Enterprise SS-12D11G5R:XKBENTERPRISESS-12D11G5R
- moved J1 1.00 mm to (61.0, 36.5)
Connections:
- new net BATT+SWITCHED: Q1.3, U$3.CENTER
- net BATT+: now also U$3.LEFT; no longer Q1.3
Routing:
- net BATT+: track 86.1 -> 83.6 mm
- net 0: track 81.0 -> 79.0 mm
- net TX: track 49.4 -> 48.4 mm
- net RX: track 57.0 -> 56.0 mm
- net CHIP_PU: track 91.3 -> 90.3 mm
- net 3.3V: track 74.6 -> 73.6 mm
Other:
- outline, holes or cut-outs redrawn
- board text added: "- 5V-8V +"
- board text removed: "5V-8V"
