File: Solar ESP Modules/Solar Power Management ESP32.sch (EAGLE design)
At the start: 35 parts, among them IC1 TP4056, IC5 1117-33, Q1 FDN360P, U2 ESP-WROOM-32NARROW

Commit message: save
Parts:
- removed D1: MBRA210LT3, microbuilder:DIODESMA
- removed R8: 1K, rcl:R-EU_R1206
- added C14, C16: 0.1uF, SparkFun:CAP0603-CAP
- added C15, C4, C5: 10uF, SparkFun:CAP_POL1206
- added D21: RED/GRN BICOLOR 3528 LED, Wurth_Elektronik_Optoelectronics_rev15c:WL-SBTW-150141RB73100-R&B
- added IC2: 1117-33, v-reg:LD117AS33TR
- added J1, J2: (no value), SparkFun-Connectors2:CONN_03X2SHROUD
- added J3: USB-C-Socket, SparkFun-Connectors:USB_C16PIN
- added R1, R21: 10k, SparkFun-Resistors:10KOHM-0603-1/10W-1%
- added R22, R27: 5.1k, SparkFun-Resistors:5.1KOHM5.1KOHM-0603-1/10W-1%
- added R30, R31: 1K, SparkFun:RESISTOR0603-RES
- added SJ1, SJ2: (no value), jumper:SJ
- added T3, T4: MBT2N2222, transistor:MMBT2222ALT1-NPN-SOT23-BEC
- added U6: FT232RLSSOP, SparkFun:FT232RLSSOP
- BZ1, BZ2, SZ1, SZ2: value 1K -> (none)
- renumbered R11 to BZ1, R12 to BZ2, R13 to SZ1, R14 to SZ2
Connections:
- removed net N$2: Q1.G, R15.2, R8.2
- new net 26_BEEPER: U2.IO26
- new net 3VUSB: C16.1, U6.3V3OUT, U6.VCCIO
- new net CC1: J3.CC1, R27.2
- new net CC2: J3.CC2, R22.2
- new net CTS: U6.CTS
- new net D+1: J3.D+, U6.USBDP
- new net D-1: J3.D-, U6.USBDM
- new net DTR: R1.1, T3.E, U6.DTR
- new net N$4: R1.2, T4.B
- new net N$6: R21.2, T3.B
- new net N$7: D21.C2, R30.2
- new net N$9: D21.C1, R31.2
- new net RTS: R21.1, T4.E, U6.RTS
- new net RXLED: R30.1, U6.RXLED
- new net SHLD: J3.SHLD
- new net TXLED: R31.1, U6.TXLED
- net 0: now also J1.6, J2.6, T3.C
- net 3.3V: now also C5.+, IC2.OUT, J1.2, J2.2
- net BATT-VOLTAGE-ADC: now also SJ2.1, SJ2.2, U2.SENSOR_VN; no longer U2.IO35
- net CHIP_PU: now also J1.1, J2.1, T4.C
- net GND: now also C14.2, C15.-, C16.2, C4.-, C5.-, IC2.ADJ, J1.4, J2.4, J3.GND, R22.1, R27.1, U6.AGND, U6.GND18, U6.GND21, U6.GND7, U6.TEST
- net RX: now also J1.3, J2.3, U6.RXD
- net SOLAR+: now also Q1.G, R15.2
- net SOLAR-VOLTAGE-ADC: now also SJ1.1, SJ1.2, U2.SENSOR_VP; no longer U2.IO34
- net TX: now also J1.5, J2.5, U6.TXD
- net VBUS: now also C14.1, C15.+, C4.+, D21.A1, D21.A2, IC2.IN, J3.VBUS, U6.VCC; no longer D1.A, R8.1
- net VCC: no longer D1.C
Other:
- note added: "AUTORESET"
- note added: "Boot Mode Configuration Pin Default Boot Download GPIO0 1 1 0 U0TXD 1 1 x GPIO2 0 x 0 GPIO4 0 x x MTDO 1 x x GPIO5 1 1 x If U0TXD, GPIO2, GPIO5 are floating, GPIO0 determines boot mode"
- note added: "If DTR is LOW, toggling RTS from HIGH to LOW resets to run mode. If RTS is HIGH, toggling DTR from LOW to HIGH resets to bootloader."
- note added: "USB TO SERIAL"
- note added: "https://www.superhouse.tv/esp-prog/"
- moved on the sheet: C2, D11

Commit message: update
Parts:
- added U$3: XKBENTERPRISESS-12D11G5R, XKB Enterprise SS-12D11G5R:XKBENTERPRISESS-12D11G5R
Connections:
- new net BATT+SWITCHED: Q1.D, U$3.CENTER
- net BATT+: now also U$3.LEFT; no longer Q1.D
Other:
- moved on the sheet: BZ1, BZ2, C12, C13, C2, C4, C5, D11, IC2, IC5, J1, J2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
