File: NODEMCU SHIELDS/untitled.brd (EAGLE design)
At the start: 100 x 100 mm, 83 parts, among them IC4 LM2596HV-5, IC6 1117-33, J6 AUDIO_JACK_3.5MM_KIT, Q10 35A/25V/8.5mΩ, Q11 200mA/40V, Q2 200mA/40V, Q3 35A/25V/8.5mΩ, Q4 35A/25V/8.5mΩ, Q5 35A/25V/8.5mΩ, Q6 35A/25V/8.5mΩ, Q7 35A/25V/8.5mΩ, Q8 35A/25V/8.5mΩ, Q9 35A/25V/8.5mΩ

Commit message: update
Parts:
- removed C3: 10uF, SparkFun:CPOL-RADIAL-10UF-25V
- removed J6: AUDIO_JACK_3.5MM_KIT, SparkFun-Connectors:AUDIO-JACK-KIT
- removed PSU-OUT: MCV3, con-phoenix-381_l:MCV3
- removed Q11: 200mA/40V, SparkFun-DiscreteSemi:TO-92
- removed R10, R8: 100k, resistor:0204/7
- removed R13: 100K, adafruit:0204/7
- removed R7: BURDEN, resistor:0204/7
- added C5: 220µF 50V, resistor:E3,5-8
- added IO0, IO12, IO14: (no value), SparkFun-Connectors:1X03_LOCK
- added STATUS: (no value), SparkFun-LED:LED_3MM
- D12: value 5.1V1SMB5918BT3G9 -> 5.1VZ
- R11: value 1K -> R-IRL
- R12: value 1K -> 150R
- moved IR1 122.1 mm to (18.0, 4.00), turned to 270 degrees
- moved R12 119.3 mm to (15.8, 9.00), turned to 0 degrees
- moved IR2 115.1 mm to (73.2, 10.0), turned to 180 degrees
- moved R11 110.7 mm to (15.8, 11.5), turned to 0 degrees
- moved S1 108.4 mm to (76.4, 13.7)
- moved R9 104.9 mm to (84.6, 18.3), turned to 90 degrees
- moved C8 81.9 mm to (86.8, 77.0), turned to 180 degrees
- moved D12 76.0 mm to (76.0, 85.0), turned to 90 degrees
- moved X2 71.3 mm to (17.0, 77.0)
- moved C2 64.0 mm to (66.0, 85.5), turned to 90 degrees
- moved IC6 63.2 mm to (76.0, 77.0), turned to 270 degrees
- moved C1 63.1 mm to (28.0, 82.5), turned to 90 degrees
- moved D39 57.2 mm to (66.0, 79.5)
- moved IC4 57.1 mm to (41.0, 83.0), turned to 90 degrees
- moved U$1 57.0 mm to (45.0, 16.0)
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Connections:
- removed net 5VREG: R11.2
- removed net IRSNDGND: IR1.K, Q11.3
- removed net N$9: Q11.2, R12.1, R13.1
- removed net REF-TENSION: C3.1, J6.SLEEVE, R10.2, R7.1, R8.1
- new net IO2_STATUS_LED: R12.2, U$1.24
- new net N$1: R12.1, STATUS.A
- new net N$2: IO0.2, U$1.25
- new net N$3: IO12.2, U$1.13
- new net N$4: IO14.2, U$1.12
- net 3.3V: now also IO0.3, IO12.3, IO14.3; no longer R8.2
- net 5V: now also C5.+, U$1.19; no longer PSU-OUT.2
- net BEEPER: now also U$1.15
- net CT-SENSOR: now also U$1.9; no longer J6.RING, J6.RSH, J6.TIP, J6.TSH, R7.2
- net DHT11: now also U$1.23
- net DIO1: now also U$1.3
- net DIO2: now also U$1.4
- net DIO3: now also U$1.5
- net DIO4: now also U$1.6
- net DIO5: now also U$1.7
- net DIO6: now also U$1.8
- net GND: now also C5.-, IO0.1, IO12.1, IO14.1, IR1.K, STATUS.K, U$1.14, U$1.32; no longer C3.2, PSU-OUT.3, Q11.1, R10.1, R13.2
- net IRRECV: now also U$1.10
- net IRSEND: now also R11.2, U$1.26; no longer R12.2
- net OUT1: now also U$1.37
- net OUT2: now also U$1.36
- net OUT3: now also U$1.33
- net OUT4: now also U$1.31
- net OUT5: now also U$1.30
- net OUT6: now also U$1.29
- net OUT7: now also U$1.28
- net OUT8: now also U$1.27
- net RF-DATA: now also U$1.11
- net VM: no longer PSU-OUT.1
Routing:
- net 3.3V: track 0.00 -> 238.3 mm
- net 5V: track 0.00 -> 191.2 mm, vias 0 -> 1
- net DIO1: track 0.00 -> 187.4 mm
- net OUT1: track 0.00 -> 179.7 mm
- net DIO2: track 0.00 -> 172.8 mm
- net OUT2: track 0.00 -> 165.5 mm
- net DIO3: track 0.00 -> 158.3 mm
- net OUT3: track 0.00 -> 146.2 mm
- net DIO4: track 0.00 -> 144.9 mm
- net DIO5: track 0.00 -> 133.3 mm
- net OUT4: track 0.00 -> 129.4 mm
- net RF-DATA: track 0.00 -> 124.8 mm
- net DIO6: track 0.00 -> 122.9 mm
- net OUT5: track 0.00 -> 115.2 mm
- net OUT6: track 0.00 -> 101.0 mm
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- added copper zone on layer 1, net 5V
- added copper zone on layer 1, net GND
- added copper zone on layer 16, net GND
- added copper zone on layer 1, net N$164
- added copper zone on layer 1, net N$41
- added copper zone on layer 1, net N$42
- added copper zone on layer 1, net N$43
- added copper zone on layer 1, net N$44
- added copper zone on layer 1, net N$45
- added copper zone on layer 1, net N$46
- added copper zone on layer 1, net N$47
- added copper zone on layer 1, net N$7
- added copper zone on layer 1, net VM
Other:
- board size 100 x 100 mm -> 90 x 90 mm
- board text added: "3.3V"
- board text added: "SIG"
- board text added: "VM"
- board text removed: "GND 5V VM"
