File: NODEMCU SHIELDS/untitled.sch (EAGLE design)
At the start: 83 parts, among them IC4 LM2596HV-5, IC6 1117-33, J6 AUDIO_JACK_3.5MM_KIT, Q10 35A/25V/8.5mΩ, Q11 200mA/40V, Q2 200mA/40V, Q3 35A/25V/8.5mΩ, Q4 35A/25V/8.5mΩ, Q5 35A/25V/8.5mΩ, Q6 35A/25V/8.5mΩ, Q7 35A/25V/8.5mΩ, Q8 35A/25V/8.5mΩ, Q9 35A/25V/8.5mΩ

Commit message: update
Parts:
- removed C3: 10uF, SparkFun:CAP_POLPTH2
- removed J6: AUDIO_JACK_3.5MM_KIT, SparkFun-Connectors:AUDIO_JACK_3.5MM_KIT
- removed PSU-OUT: MCV3, con-phoenix-381_l:MCV3
- removed Q11: 200mA/40V, SparkFun-DiscreteSemi:TRANS_NPN-2N3904
- removed R10, R8: 100k, resistor:R-US_0204/7
- removed R13: 100K, adafruit:R-US_0204/7
- removed R7: BURDEN, resistor:R-US_0204/7
- added C5: 220µF 50V, resistor:CPOL-EUE3.5-8
- added IO0, IO12, IO14: (no value), SparkFun-Connectors:CONN_03LOCK
- added STATUS: (no value), SparkFun-LED:LED3MM
- D12: value 5.1V1SMB5918BT3G9 -> 5.1VZ
- R11: value 1K -> R-IRL
- R12: value 1K -> 150R
Connections:
- removed net 5VREG: R11.2
- removed net IRSNDGND: IR1.C, Q11.C
- removed net N$9: Q11.B, R12.1, R13.1
- removed net REF-TENSION: C3.+, J6.SLEEVE, R10.2, R7.1, R8.1
- new net IO2_STATUS_LED: R12.2, U$1.IO2
- new net N$1: R12.1, STATUS.A
- new net N$2: IO0.2, U$1.IO0
- new net N$3: IO12.2, U$1.IO12
- new net N$4: IO14.2, U$1.IO14
- net 3.3V: now also IO0.3, IO12.3, IO14.3; no longer R8.2
- net 5V: now also C5.+, U$1.5V; no longer PSU-OUT.2.SK
- net BEEPER: now also U$1.IO13
- net CT-SENSOR: now also U$1.IO25; no longer J6.RING, J6.RSH, J6.TIP, J6.TSH, R7.2
- net DHT11: now also U$1.IO15
- net DIO1: now also U$1.SVP
- net DIO2: now also U$1.SVN
- net DIO3: now also U$1.IO34
- net DIO4: now also U$1.IO35
- net DIO5: now also U$1.IO32
- net DIO6: now also U$1.IO33
- net GND: now also C5.-, IO0.1, IO12.1, IO14.1, IR1.C, STATUS.C, U$1.GND@14, U$1.GND@32; no longer C3.-, PSU-OUT.3.SK, Q11.E, R10.1, R13.2
- net IRRECV: now also U$1.IO26
- net IRSEND: now also R11.2, U$1.IO4; no longer R12.2
- net OUT1: now also U$1.IO23
- net OUT2: now also U$1.IO22
- net OUT3: now also U$1.IO21
- net OUT4: now also U$1.IO19
- net OUT5: now also U$1.IO18
- net OUT6: now also U$1.IO5
- net OUT7: now also U$1.IO17
- net OUT8: now also U$1.IO16
- net RF-DATA: now also U$1.IO27
- net VM: no longer PSU-OUT.1.SK
Other:
- moved on the sheet: R12, U$1
