File: WS2812 panels/60 LED panel with ESP01/80 LED WS2812 panels.brd (EAGLE design)
At the start: 100 x 100 mm, 153 parts, among them IC4 LM2596-5S, Q3 BSS138, U4 1117/3.3v

Commit message: DB board
Parts:
- removed C1, C2: 220uF, cutout capacitor:CAPACITOR-SIDEWAY-CUTOUT
- removed ESP: ESP01, esp8266modules:ESP01
- removed S1: RST, SparkFun-Switches:TACTILE_SWITCH_PTH_6.0MM_KIT
- removed S2: IO0, SparkFun-Switches:TACTILE_SWITCH_PTH_6.0MM_KIT
- added 2, 3V3, A0, GND: TPTP13SQ, testpad:TP13SQ
- added C61: 0.1UF, rcl:C1206@1
- added C62, C63: 220uF, rcl:E3,5-10
- added C64: 22UF, rcl:C1812K@1
- added D61: SS34, diode:DO-214AC
- added D62: 1N4148, SparkFun-DiscreteSemi:SOD-323
- added IC1: TP4056, TP4056:SOP-8
- added IC2: PC817, optocoupler:DIL04
- added IC3: ESP8266_ESP-12, ESP8266-ESP12:ESP8266-ESP12
- added LED1: RED, led:LED3MM
- added LED2: GREEN, led:LED3MM
- added MODE0, RESET: TACTSW R/A 6x6x8MM, dp_devices:SW_TACT_STANDARD_RIGHT_ANGLE
- added R10, R9: 1K, rcl:R1206
- added R11: 1K, resistor:R1206
- added R12, R4: 10K, resistor:R1206
- added R5: 2K, resistor:R1206
- added R6: 100, rcl:R1206
- added R7, R8: 2K, rcl:R1206
- added SJ6: (no value), jumper:SJ_2
- added U$1: FS312F-G, buckboost:SOT23-6
- added U$13: JRC-21F-4100, JRC-21F:JRC-21F-4100
- added U$2: FS8205, buckboost:SOT23-6
- added U$3: XKBENTERPRISESS-12D11G5R, XKB Enterprise SS-12D11G5R:XKBENTERPRISESS-12D11G5R
- added X3, X5: (no value), con-wago-500:W237-102
- C10, C11, C12, C13, C14, C15, C16, C17, C18, C19, C20, C21, C22, C23, C24, C25, C26, C27, C28, C29, C3, C30, C31, C32, C33, C34, C35, C36, C37, C38, C39, C4, C40, C41, C42, C43, C44, C45, C46, C47, C48, C49, C5, C50, C51, C52, C53, C54, C55, C56, C6, C7, C8, C9: device rcl:C1206 -> rcl:C1206@1
- R1: device SparkFun-Resistors:1206 -> resistor:R1206
- R2, R3: value 10k -> 10K; device SparkFun-Resistors:1206 -> resistor:R1206
- RX, TX: value (none) -> TPTP13SQ; device wirepad:2,15/1,0 -> testpad:TP13SQ
- moved R1 53.1 mm to (73.5, 19.0), turned to 90 degrees
- moved TX 50.5 mm to (54.0, 31.0), flipped to the bottom
- moved RX 49.8 mm to (54.0, 34.0), flipped to the bottom
- moved R2 38.5 mm to (65.0, 29.0)
- moved R3 35.4 mm to (65.0, 33.0), turned to 180 degrees
- moved C60 34.5 mm to (35.0, 28.0)
- moved U4 31.1 mm to (12.0, 34.5), turned to 270 degrees
- moved C58 27.7 mm to (11.5, 29.0)
- moved C59 26.2 mm to (19.0, 28.0), turned to 180 degrees
- moved C57 22.0 mm to (27.0, 28.0)
- moved R23 18.4 mm to (27.0, 34.0), turned to 90 degrees
- moved L1 18.1 mm to (52.0, 7.50)
- moved IC4 17.0 mm to (68.0, 7.00)
- moved Q3 16.4 mm to (22.5, 34.0), turned to 90 degrees
- moved C48 16.0 mm to (10.0, 51.0)
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Connections:
- removed net 5V: R25.1
- removed net IO0: ESP.GPIO0, R2.2, S2.1
- removed net IO2: ESP.GPIO2, Q3.2, R23.2
- removed net PD: ESP.CH_PD, R3.1
- removed net RST: ESP.RST, R1.2, S1.1
- new net 5VREG: C63.+, D61.A, D62.C, IC4.4, L1.2, U$13.COIL-, U$13.NO, U$3.RIGHT
- new net ADC: A0.TP, IC3.10
- new net BATT+: IC1.5, R6.2, U$13.NC, U$3.LEFT, X5.2
- new net BATT-: C61.1, U$1.6, U$2.1, X5.1
- new net CHG: IC1.7, R10.2
- new net EXTGPIO: IC3.5
- new net IO0/AUX1-INPUT: IC3.4, MODE0.1, R3.2
- new net LEDCHR: LED1.K, R10.1
- new net LEDSBY: LED2.K, R9.1
- new net N$55: IC2.1, R5.1
- new net N$56: 2.TP, IC3.3, R2.2
- new net N$57: R7.2, U$1.2
- new net N$58: IC3.12, SJ6.1
- new net N$59: IC3.11, R11.1
- new net N$60: IC3.2, R12.2
- new net N$61: R4.1, SJ6.3
- new net OC: U$1.3, U$2.4
- new net OD: U$1.1, U$2.6
- new net OPTO: IC2.4, IC3.6, R1.1
- new net PROG: IC1.2, R8.1
- new net RELAY1: IC3.14
- new net RESET: IC3.9, RESET.1, SJ6.2
- new net STANDBY: IC1.6, R9.2
- new net STATUSLED: IC3.15
- new net VCC-PROT: C61.2, R6.1, U$1.5
- new net VUSB: C64.1, D61.C, IC1.4, IC1.8, LED1.A, LED2.A
- new net WS2812-SIG: IC3.13, Q3.2, R23.2
- net +3V3: now also 3V3.TP, IC3.16, R1.2, R11.2, R3.1, R4.2; no longer ESP.VCC, R1.1, R2.1, R3.2
- net GND: now also C62.-, C63.-, C64.2, D62.A, GND.TP, IC1.1, IC1.3, IC2.2, IC2.3, IC3.1, MODE0.2, R12.1, R2.1, R7.1, R8.2, RESET.2, U$13.COIL+, U$2.3, X3.1; no longer C1.-, C2.-, ESP.GND, S1.3, S2.3
- net HI-V-IN: now also C62.+, R5.2; no longer C1.+
- net LED1PWR: now also R25.1, U$13.C1, U$13.C2, U$3.CENTER, X3.2; no longer C2.+, IC4.4, L1.2
- net RX: now also IC3.8, RX.TP; no longer ESP.RX, RX.1
- net TX: now also IC3.7, TX.TP; no longer ESP.TX, TX.1
Routing:
- net RESET: track 0.00 -> 66.4 mm
- net IO0/AUX1-INPUT: track 0.00 -> 58.4 mm, vias 0 -> 2
- net LED1PWR: track 0.00 -> 49.0 mm, vias 0 -> 14
- net PD: track 37.7 -> 0.00 mm
- net IO2: track 37.4 -> 0.00 mm
- net +3V3: track 74.3 -> 110.6 mm
- net IO0: track 34.4 -> 0.00 mm
- net OPTO: track 0.00 -> 33.4 mm
- net WS2812-SIG: track 0.00 -> 29.9 mm, vias 0 -> 2
- net DIN1: track 110.5 -> 83.6 mm
- net RST: track 26.8 -> 0.00 mm, vias 1 -> 0
- net TX: track 25.3 -> 0.00 mm
- net VUSB: track 0.00 -> 24.2 mm
- net RX: track 18.0 -> 0.00 mm
- net N$58: track 0.00 -> 15.2 mm
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- added copper zone on layer 1, net 5VREG
- added copper zone on layer 1, net BATT+
- added copper zone on layer 1, net BATT-
- added copper zone on layer 1, net VUSB
- removed copper zone on layer 1, net GND
Other:
- outline, holes or cut-outs redrawn
- board text added: "1"
- board text added: "10"
- board text added: "11"
- board text added: "20"
- board text added: "21"
- board text added: "30"
- board text added: "31"
- board text added: "40\"
- board text added: "41"
- board text added: "50"
- board text added: "51"
- board text added: "5V UPS OUTPUT"
- board text added: "60"
- board text added: "7-35V INPUT"
- board text added: "LIPO BATT"
- board text added: "RUN/SLP"
