File: WS2812 panels/60 LED panel with ESP01/80 LED WS2812 panels.sch (EAGLE design)
At the start: 153 parts, among them IC4 LM2596-5S, Q3 BSS138, U4 1117/3.3v

Commit message: DB board
Parts:
- removed C1, C2: 220uF, cutout capacitor:CAPACITOR-SIDEWAY-CUTOUT
- removed ESP: ESP01, esp8266modules:ESP01
- removed S1: RST, SparkFun-Switches:MOMENTARY-SWITCH-SPST-PTH-6.0MM-KIT
- removed S2: IO0, SparkFun-Switches:MOMENTARY-SWITCH-SPST-PTH-6.0MM-KIT
- added 2, 3V3, A0, GND: TPTP13SQ, testpad:TPTP13SQ
- added C61: 0.1UF, rcl:C-EUC1206
- added C62, C63: 220uF, rcl:CPOL-EUE3.5-10
- added C64: 22UF, rcl:C-EUC1812K
- added D61: SS34, diode:DIODE-DO-214AC
- added D62: 1N4148, SparkFun-DiscreteSemi:DIODE-BAS16J
- added IC1: TP4056, TP4056:TP4056
- added IC2: PC817, optocoupler:PC817
- added IC3: ESP8266_ESP-12, ESP8266-ESP12:ESP8266_ESP-12
- added LED1: RED, led:LED3MM
- added LED2: GREEN, led:LED3MM
- added MODE0, RESET: TACTSW R/A 6x6x8MM, dp_devices:SW_TACT_4P_B
- added R10, R9: 1K, rcl:R-EU_R1206
- added R11: 1K, resistor:R-US_R1206
- added R12, R4: 10K, resistor:R-US_R1206
- added R5: 2K, resistor:R-US_R1206
- added R6: 100, rcl:R-EU_R1206
- added R7, R8: 2K, rcl:R-EU_R1206
- added SJ6: (no value), jumper:SJ2W
- added U$1: FS312F-G, buckboost:FS312F-G
- added U$13: JRC-21F-4100, JRC-21F:JRC-21F-4100
- added U$2: FS8205, buckboost:FS8205
- added U$3: XKBENTERPRISESS-12D11G5R, XKB Enterprise SS-12D11G5R:XKBENTERPRISESS-12D11G5R
- added X3, X5: (no value), con-wago-500:W237-102
- R1: device SparkFun-Resistors:10OHM-1206-1/4W-1% -> resistor:R-US_R1206
- R2, R3: value 10k -> 10K; device SparkFun-Resistors:10OHM-1206-1/4W-1% -> resistor:R-US_R1206
- RX, TX: value (none) -> TPTP13SQ; device wirepad:2,15/1,0 -> testpad:TPTP13SQ
Connections:
- removed net 5V: R25.1
- removed net IO0: ESP.GPIO0, R2.2, S2.1
- removed net IO2: ESP.GPIO2, Q3.S, R23.2
- removed net PD: ESP.CH_PD, R3.1
- removed net RST: ESP.RST, R1.2, S1.1
- new net 5VREG: C63.+, D61.A, D62.C, IC4.FB, L1.2, U$13.COIL-, U$13.NO, U$3.RIGHT
- new net ADC: A0.TP, IC3.ADC
- new net BATT+: IC1.BAT, R6.2, U$13.NC, U$3.LEFT, X5-2.KL
- new net BATT-: C61.1, U$1.GND, U$2.S1, X5-1.KL
- new net CHG: IC1.CHRG, R10.2
- new net EXTGPIO: IC3.GPIO5
- new net IO0/AUX1-INPUT: IC3.GPIO0, MODE0.1, R3.2
- new net LEDCHR: LED1.C, R10.1
- new net LEDSBY: LED2.C, R9.1
- new net N$55: IC2.A, R5.1
- new net N$56: 2.TP, IC3.GPIO2, R2.2
- new net N$57: R7.2, U$1.CS
- new net N$58: IC3.GPIO16, SJ6.1
- new net N$59: IC3.CH_PD, R11.1
- new net N$60: IC3.GPIO15, R12.2
- new net N$61: R4.1, SJ6.3
- new net OC: U$1.OC, U$2.G2
- new net OD: U$1.OD, U$2.G1
- new net OPTO: IC2.COL, IC3.GPIO4, R1.1
- new net PROG: IC1.PROG, R8.1
- new net RELAY1: IC3.GPIO12
- new net RESET: IC3.REST, RESET.1, SJ6.2
- new net STANDBY: IC1.STDBY, R9.2
- new net STATUSLED: IC3.GPIO13
- new net VCC-PROT: C61.2, R6.1, U$1.VCC
- new net VUSB: C64.1, D61.C, IC1.CE, IC1.VCC, LED1.A, LED2.A
- new net WS2812-SIG: IC3.GPIO14, Q3.S, R23.2
- net +3V3: now also 3V3.TP, IC3.VCC, R1.2, R11.2, R3.1, R4.2; no longer ESP.VCC, R1.1, R2.1, R3.2
- net GND: now also C62.-, C63.-, C64.2, D62.A, GND.TP, IC1.GND, IC1.TEMP, IC2.C, IC2.EMIT, IC3.GND, MODE0.2, R12.1, R2.1, R7.1, R8.2, RESET.2, U$13.COIL=, U$2.S2, X3-1.KL; no longer C1.-, C2.-, ESP.GND, S1.2, S2.2
- net HI-V-IN: now also C62.+, R5.2; no longer C1.+
- net LED1PWR: now also R25.1, U$13.C, U$3.CENTER, X3-2.KL; no longer C2.+, IC4.FB, L1.2
- net RX: now also IC3.TXD, RX.TP; no longer ESP.RXD, RX.P
- net TX: now also IC3.RXD, TX.TP; no longer ESP.TXD, TX.P
Other:
- note added: "+"
- note added: "-"
- moved on the sheet: R1, R2, R3
