File: 5V StepDown PCB/5V Stepdown.brd (EAGLE design)
At the start: 98.9 x 98.9 mm, 29 parts, among them IC1 LM2596HV-5

Commit message: PCB5102 Board
Parts:
- removed C25, C33: 10uF, A9G:DISCRETE_C1206
- removed C32, C34, C48: 0.1uF, A9G:DISCRETE_C0603
- removed D10: SS34, diode:DO-214AC
- removed D11, D12, D7, D8, D9: WS2812B, SparkFun-LED:WS2812B
- added C10: 104, rcl:C1206
- added C11: 20p, z_jlc_smt:1206
- added C12, C13, C14, C15, C16: 104, z_jlc_smt:1206
- added C37: 10uF, SparkFun:EIA3216
- added CONN2, CONN3: WJ212R-THR-3.5-4, WJ212R-THR-3.5-3.81:WJ212R-THR-3.5-4
- added IC2, IC3: LM2596HV-5, linear:TO263-5
- added L2, L3: 33uH, inductors:DR127
- added LED1: (no value), led:LED3MM
- added R1, R2, R30, R32: 75K, adafruit:M1206
- added R3, R33, R34, R4: 49.9K, adafruit:M1206
- added R6: 715R, z_jlc_smt:1206
- added R7: 330, z_jlc_smt:1206
- added R9: 10K, z_jlc_smt:1206
- added SD1: TF-HOLDER, sd-mmc:TF-PULL
- added U$1, U$2: TPS2514, TPS2514:TPS2514
- added U$3, U$4: USB+SHIELDUSB-A-S-NOSILK-FEMALE, SparkFun-Connectors:USB-A-S-NOSILK-FEMALE
- added U1: GL827L150MIL, xmgu2008:SSOP28-39
- added X1, X3: (no value), con-berg:PN87520
- added X2: USBPCB, SparkFun:USB-A-PCB
- added Y1: 12M, xmgu2008:HC49US
- C3, C4, C5, C6: value 0.1uF -> 220µF 50V; device A9G:DISCRETE_C0603 -> resistor:PANASONIC_E
- C7: value 0.1uF -> 104; device A9G:DISCRETE_C0603 -> rcl:C1206
- C8: value 0.1uF -> 10uF; device A9G:DISCRETE_C0603 -> SparkFun:EIA3216
- C9: value 0.1uF -> 20p; device A9G:DISCRETE_C0603 -> z_jlc_smt:1206
- D3, D5: value WS2812B -> SS34; device SparkFun-LED:WS2812B -> semicon-smd-ipc:SOD87
- D4, D6: value WS2812B -> SMB3Z5.1A; device SparkFun-LED:WS2812B -> diode:SMB
- moved C9 288.8 mm to (58.4, 92.5), turned to 90 degrees
- moved C6 224.1 mm to (27.5, 79.5), turned to 90 degrees
- moved C5 213.5 mm to (36.5, 79.5), turned to 90 degrees
- moved D6 205.6 mm to (27.5, 70.5)
- moved D5 194.9 mm to (35.5, 70.5), turned to 180 degrees
- moved C4 188.8 mm to (5.50, 79.5), turned to 90 degrees
- moved C8 186.9 mm to (2.00, 20.0), turned to 270 degrees
- moved C7 185.8 mm to (10.0, 30.0)
- moved C3 177.4 mm to (14.5, 79.5), turned to 90 degrees
- moved D4 170.0 mm to (5.50, 70.5)
- moved D3 158.6 mm to (13.5, 70.5), turned to 180 degrees
- moved CONN1 80.9 mm to (56.1, 35.9), turned to 270 degrees
- moved D1 76.8 mm to (75.5, 38.5), turned to 180 degrees
- moved C1 75.2 mm to (87.5, 39.5), turned to 180 degrees
- moved L1 69.6 mm to (75.5, 28.5), turned to 270 degrees
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Connections:
- removed net 5VRGBLED: C25.2, C3.2, C32.2, C33.2, C34.2, C4.2, C48.2, C5.2, C6.2, C7.2, C8.2, C9.2, D10.C, D11.1, D12.1, D3.1, D4.1, D5.1, D6.1, D7.1, D8.1, D9.1
- removed net GND_BOTTOM: C1.-, C2.-, CONN1.2A, CONN1.2B, CONN1.4A, CONN1.4B, D1.2, D2.A, IC1.3, IC1.5, IC1.6
- removed net IO48/RGBLED: D8.4
- removed net N$11: D11.4, D7.2
- removed net N$12: D11.2, D12.4
- removed net N$3: D3.4, D9.2
- removed net N$4: D3.2, D4.4
- removed net N$7: D8.2, D9.4
- removed net N$8: D4.2, D5.4
- removed net N$9: D5.2, D6.4
- new net CARD1_3V3_CARD1: C14.1, C15.1, U1.11, U1.3, U1.7
- new net CARD1_ACCESS: R7.2, U1.28
- new net CARD1_CD: SD1.9, U1.15
- new net CARD1_CLK: SD1.5, U1.20
- new net CARD1_CMD: SD1.3, U1.22
- new net CARD1_D0: SD1.7, U1.17
- new net CARD1_D1: SD1.8, U1.16
- new net CARD1_D2: SD1.1, U1.25
- new net CARD1_D3: SD1.2, U1.24
- new net CARD1_SD_VDD: C16.1, SD1.4, U1.2
- new net D+: R2.2, R3.2, R32.2, R33.2, U$1.DP1, U$2.DP1, U$3.D+, U$4.D+, X1.3, X3.3
- new net D-: R1.2, R30.2, R34.2, R4.2, U$1.DM1, U$2.DM1, U$3.D-, U$4.D-, X1.2, X3.2
- new net DM1: U1.9, X2.USB_M
- new net DP1: U1.8, X2.USB_P
- new net N$2: C9.2, U1.4, Y1.2
- new net N$21: C12.1, U1.13
- new net N$26: LED1.A, R7.1
- new net N$28: R9.1, U1.14
- new net N$5: C11.2, U1.5, Y1.1
- new net SW-L1: D3.1, IC2.2, L2.1
- new net SW-L2: D5.1, IC3.2, L3.1
- net +24V: now also C3.+, C5.+, CONN2.3A, CONN2.3B, CONN3.3A, CONN3.3B, IC2.1, IC3.1
- net 5V: now also C13.1, U1.12, X2.5V; no longer D10.A
- net 5V-REG: now also C10.1, C37.A, C4.+, C6.+, C7.1, C8.A, CONN2.1A, CONN2.1B, CONN3.1A, CONN3.1B, D4.C, D6.C, IC2.4, IC3.4, L2.2, L3.2, R1.1, R2.1, R30.1, R32.1, U$1.IN, U$2.IN, U$3.VBUS, U$4.VBUS, X1.1, X3.1
- net GND: now also C1.-, C10.2, C11.1, C12.2, C13.2, C14.2, C15.2, C16.2, C2.-, C3.-, C37.C, C4.-, C5.-, C6.-, C7.2, C8.C, CONN1.2A, CONN1.2B, CONN1.4A, CONN1.4B, CONN2.2A, CONN2.2B, CONN2.4A, CONN2.4B, CONN3.2A, CONN3.2B, CONN3.4A, CONN3.4B, D1.2, D2.A, D3.2, D4.A, D5.2, D6.A, IC1.3, IC1.5, IC1.6, IC2.3, IC2.5, IC2.6, IC3.3, IC3.5, IC3.6, LED1.K, R3.1, R33.1, R34.1, R4.1, R6.1, R9.2, SD1.6, SD1.S1, SD1.S2, SD1.S3, SD1.S4, U$1.GND, U$2.GND, U$3.GND, U$3.S1, U$3.S2, U$4.GND, U$4.S1, U$4.S2, U1.6, X1.4, X2.GND, X3.4; no longer C25.1, C3.1, C32.1, C33.1, C34.1, C4.1, C48.1, C5.1, C6.1, C7.1, C8.1, D11.3, D12.3, D3.3, D4.3, D5.3, D6.3, D7.3, D8.3, D9.3
- net N$10: now also R6.2, U1.10; no longer D6.2, D7.4
Routing:
- net 5V-REG: track 0.00 -> 50.6 mm, vias 0 -> 5
- net D+: track 0.00 -> 33.8 mm
- net D-: track 0.00 -> 32.3 mm
- net CARD1_3V3_CARD1: track 0.00 -> 30.8 mm
- net 5V: track 0.00 -> 26.7 mm, vias 0 -> 2
- net DP1: track 0.00 -> 25.8 mm, vias 0 -> 2
- net DM1: track 0.00 -> 25.1 mm, vias 0 -> 2
- net CARD1_SD_VDD: track 0.00 -> 24.1 mm, vias 0 -> 2
- net N$5: track 0.00 -> 22.9 mm, vias 1 -> 0
- net N$2: track 0.00 -> 20.3 mm, vias 1 -> 0
- net GND: track 0.00 -> 16.2 mm, vias 0 -> 68
- net LINK3: track 0.00 -> 14.0 mm, vias 0 -> 2
- net CARD1_ACCESS: track 0.00 -> 7.88 mm
- net N$10: track 0.00 -> 6.82 mm
- net N$28: track 0.00 -> 6.58 mm
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- added copper zone on layer 1, net GND
- added copper zone on layer 16, net GND
- added copper zone on layer 1, net SW-L1
- added copper zone on layer 1, net SW-L2
- removed copper zone on layer 1, net GND_BOTTOM
Other:
- board size 98.9 x 98.9 mm -> 100 x 100 mm
- board text added: "+"
- board text added: "-"
- board text added: "5V"
- board text added: "MICROSD READER"
- board text added: "todo max2323 todo karkas throttle (soos multimeter selector pcb met spoed) Drill Batt Solar Charger Multi relay mains RJ45 WS2812s"
- board text added: "|PvdW|"
