File: 5V StepDown PCB/5V Stepdown.sch (EAGLE design)
At the start: 29 parts, among them IC1 LM2596HV-5

Commit message: PCB5102 Board
Parts:
- removed C25, C33: 10uF, A9G:DISCRETE_C-1206
- removed C32, C34, C48: 0.1uF, A9G:DISCRETE_C-0603
- removed D10: SS34, diode:DIODE-DO-214AC
- removed D11, D12, D7, D8, D9: WS2812B, SparkFun-LED:WS2812B
- added C10: 104, rcl:C-EUC1206
- added C11: 20p, z_jlc_smt:CAP1206
- added C12, C13, C14, C15, C16: 104, z_jlc_smt:CAP1206
- added C37: 10uF, SparkFun:CAP_POL1206
- added CONN2, CONN3: WJ212R-THR-3.5-4, WJ212R-THR-3.5-3.81:WJ212R-THR-3.5-4
- added IC2, IC3: LM2596HV-5, linear:LM2596S
- added L2, L3: 33uH, inductors:DR127
- added LED1: (no value), led:LED3MM
- added R1, R2, R30, R32: 75K, adafruit:R-US_M1206
- added R3, R33, R34, R4: 49.9K, adafruit:R-US_M1206
- added R6: 715R, z_jlc_smt:RESISTOR1206
- added R7: 330, z_jlc_smt:RESISTOR1206
- added R9: 10K, z_jlc_smt:RESISTOR1206
- added SD1: TF-HOLDER, sd-mmc:TF-HOLDER
- added U$1, U$2: TPS2514, TPS2514:TPS2514
- added U$3, U$4: USB+SHIELDUSB-A-S-NOSILK-FEMALE, SparkFun-Connectors:USB+SHIELDUSB-A-S-NOSILK-FEMALE
- added U1: GL827L150MIL, xmgu2008:GL827L150MIL
- added X1, X3: (no value), con-berg:PN87520
- added X2: USBPCB, SparkFun:USBPCB
- added Y1: 12M, xmgu2008:CRYSTAL2HC49US
- C3, C4, C5, C6: value 0.1uF -> 220µF 50V; device A9G:DISCRETE_C-0603 -> resistor:CPOL-EUE
- C7: value 0.1uF -> 104; device A9G:DISCRETE_C-0603 -> rcl:C-EUC1206
- C8: value 0.1uF -> 10uF; device A9G:DISCRETE_C-0603 -> SparkFun:CAP_POL1206
- C9: value 0.1uF -> 20p; device A9G:DISCRETE_C-0603 -> z_jlc_smt:CAP1206
- D3, D5: value WS2812B -> SS34; device SparkFun-LED:WS2812B -> semicon-smd-ipc:D-SOD-87
- D4, D6: value WS2812B -> SMB3Z5.1A; device SparkFun-LED:WS2812B -> diode:ZENER-DIODESMB
Connections:
- removed net 5VRGBLED: C25.2, C3.2, C32.2, C33.2, C34.2, C4.2, C48.2, C5.2, C6.2, C7.2, C8.2, C9.2, D10.C, D11.VDD, D12.VDD, D3.VDD, D4.VDD, D5.VDD, D6.VDD, D7.VDD, D8.VDD, D9.VDD
- removed net GND_BOTTOM: C1.-, C2.-, CONN1.P$2, CONN1.P$4, D1.A, D2.A, IC1.EN, IC1.GND, IC1.GND@1
- removed net IO48/RGBLED: D8.DI
- removed net N$11: D11.DI, D7.DO
- removed net N$12: D11.DO, D12.DI
- removed net N$3: D3.DI, D9.DO
- removed net N$4: D3.DO, D4.DI
- removed net N$7: D8.DO, D9.DI
- removed net N$8: D4.DO, D5.DI
- removed net N$9: D5.DO, D6.DI
- new net CARD1_3V3_CARD1: C14.1, C15.1, U1.AVDD, U1.DVDD, U1.DVDD@11
- new net CARD1_ACCESS: R7.2, U1.IO0
- new net CARD1_CD: SD1.!CARD, U1.SD_CDZ
- new net CARD1_CLK: SD1.CLK(SCLK), U1.SD_CLK
- new net CARD1_CMD: SD1.CMD(DI), U1.SD_CMD
- new net CARD1_D0: SD1.DAT0(DO), U1.D0
- new net CARD1_D1: SD1.DAT1, U1.D1
- new net CARD1_D2: SD1.DAT2, U1.D2
- new net CARD1_D3: SD1.CD/DAT3(!CS!), U1.D3
- new net CARD1_SD_VDD: C16.1, SD1.VDD, U1.PMOSO
- new net D+: R2.2, R3.2, R32.2, R33.2, U$1.DP1, U$2.DP1, U$3.D+, U$4.D+, X1.3, X3.3
- new net D-: R1.2, R30.2, R34.2, R4.2, U$1.DM1, U$2.DM1, U$3.D-, U$4.D-, X1.2, X3.2
- new net DM1: U1.DM, X2.D-
- new net DP1: U1.DP, X2.D+
- new net N$2: C9.2, U1.X1, Y1.2
- new net N$21: C12.1, U1.RST
- new net N$26: LED1.A, R7.1
- new net N$28: R9.1, U1.SD_WP
- new net N$5: C11.2, U1.X2, Y1.1
- new net SW-L1: D3.C, IC2.OUT, L2.1
- new net SW-L2: D5.C, IC3.OUT, L3.1
- net +24V: now also C3.+, C5.+, CONN2.P$3, CONN3.P$3, IC2.IN, IC3.IN
- net 5V: now also C13.1, U1.VP5, X2.VBUS; no longer D10.A
- net 5V-REG: now also C10.1, C37.+, C4.+, C6.+, C7.1, C8.+, CONN2.P$1, CONN3.P$1, D4.C, D6.C, IC2.FB, IC3.FB, L2.2, L3.2, R1.1, R2.1, R30.1, R32.1, U$1.IN, U$2.IN, U$3.VBUS, U$4.VBUS, X1.1, X3.1
- net GND: now also C1.-, C10.2, C11.1, C12.2, C13.2, C14.2, C15.2, C16.2, C2.-, C3.-, C37.-, C4.-, C5.-, C6.-, C7.2, C8.-, CONN1.P$2, CONN1.P$4, CONN2.P$2, CONN2.P$4, CONN3.P$2, CONN3.P$4, D1.A, D2.A, D3.A, D4.A, D5.A, D6.A, IC1.EN, IC1.GND, IC1.GND@1, IC2.EN, IC2.GND, IC2.GND@1, IC3.EN, IC3.GND, IC3.GND@1, LED1.C, R3.1, R33.1, R34.1, R4.1, R6.1, R9.2, SD1.S1, SD1.S2, SD1.S3, SD1.S4, SD1.VSS, U$1.GND, U$2.GND, U$3.GND, U$3.S1, U$3.S2, U$4.GND, U$4.S1, U$4.S2, U1.GND, X1.4, X2.GND, X3.4; no longer C25.1, C3.1, C32.1, C33.1, C34.1, C4.1, C48.1, C5.1, C6.1, C7.1, C8.1, D11.VSS, D12.VSS, D3.VSS, D4.VSS, D5.VSS, D6.VSS, D7.VSS, D8.VSS, D9.VSS
- net N$10: now also R6.2, U1.RREF; no longer D6.DO, D7.DI
Other:
- note removed: "POWER"
- note removed: "VIN > 5V"
