File: I2S Audio Board/pcm5102_dac.brd (EAGLE design)
At the start: 100 x 100 mm, 61 parts, among them CON3 USB-C-Socket, IC1 PCM510xA, IC4 LM2596HV-5, IC5 AP2114H-3.3TRG1, J2 AUDIO_JACK_3.5MM_PTH, U3 ESP32S3WROOM1N8R8

Commit message: PCN5102 board
Parts:
- removed DE-EMPHASIS, LATENCY: (no value), SparkFun-Connectors2:1X03_LOCK
- removed I2C, VIN: WJ212R-THR-3.5-2, WJ212R-THR-3.5-3.81:WJ212R-THR-3.5-2
- removed I2CLCD: MOLEX_SL_04-70555, molex-sl-connectors_jw:SL_70555_4
- removed IO0: MOMENTARY-SWITCH-SPST-PTH-6.0MM, SparkFun-Switches:TACTILE_SWITCH_PTH_6.0MM
- removed R22: 10K, discrete:R0603
- removed SPI: WJ212R-THR-3.5-3, WJ212R-THR-3.5-3.81:WJ212R-THR-3.5-3
- added CON7, CON8: PCB-2M3, Screw Terminals:PCB2-M3
- added D16: M4, diode:DO-214AC
- added DEMP, LAT: (no value), jumper:SJ_2
- added J1, J4, J5, J6: (no value), SparkFun-Connectors:2X5-SHROUDED
- added MODE: MOMENTARY-SWITCH-SPST-PTH-6.0MM, SparkFun-Switches:TACTILE_SWITCH_PTH_6.0MM
- added PWRIN, SWOUT: Phoenix Pluggable 5.08mm 2 way, con-phoenix-508:MSTBA2
- added Q5: NCHAN, Cohesion_parts:D-PAK_TO252AA
- added R24: 10K, SparkFun-Resistors:0603@1
- added R62: 10R, resistor:R0603
- added R63: 100K, resistor:R0603
- C42: value 10uF 50V -> 10uF
- R16: device discrete:R0603 -> SparkFun-Resistors:0603@1
- moved C24 68.7 mm to (36.0, 26.5), turned to 90 degrees
- moved R11 60.8 mm to (86.5, 18.5), turned to 270 degrees
- moved D14 60.0 mm to (35.6, 34.0), turned to 180 degrees
- moved R8 58.1 mm to (81.5, 18.5), turned to 270 degrees
- moved R10 58.0 mm to (79.0, 18.5), turned to 270 degrees
- moved C25 56.6 mm to (96.1, 39.1), turned to 90 degrees
- moved D7 56.1 mm to (17.0, 17.0), turned to 270 degrees
- moved R9 55.9 mm to (84.0, 18.5), turned to 270 degrees
- moved L5 55.2 mm to (24.5, 28.5), turned to 90 degrees
- moved C2 54.1 mm to (92.1, 18.3), turned to 0 degrees
- moved C21 51.0 mm to (57.7, 12.5)
- moved D39 50.3 mm to (20.5, 17.0), turned to 270 degrees
- moved C8 50.1 mm to (96.1, 30.1), turned to 90 degrees
- moved R1 50.0 mm to (57.7, 10.0)
- moved CON3 50.0 mm to (55.0, 7.67)
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Connections:
- new net IO1: J4.10, U3.39
- new net IO14_NEXT: J4.6, U3.22
- new net IO15_LCD_D5: J5.8, U3.8
- new net IO16_LCD_D6: J5.9, U3.9
- new net IO17_LCD_D7: J5.10, U3.10
- new net IO18_PREV: J6.5, U3.11
- new net IO2: J4.9, U3.38
- new net IO21_SHUFFLE: J4.5, U3.23
- new net IO35: J1.7, U3.28
- new net IO36: J1.6, U3.29
- new net IO37: J1.5, U3.30
- new net IO38_MOSFET: R62.1, U3.31
- new net IO45_LCD_BACKLIGHT: J1.8, U3.26
- new net IO46_PAUSE: J6.7, U3.16
- new net IO47_VOLM: J1.10, U3.24
- new net IO48_VOLP: J1.9, U3.25
- new net IO5_LCD_RS: J5.5, U3.5
- new net IO6_LCD_E: J5.6, U3.6
- new net IO7_LCD_D4: J5.7, U3.7
- new net IO8_PLAY: J6.6, U3.12
- new net IO9_STOP: J6.8, U3.17
- new net MOSFET-GND: D16.A, Q5.4, SWOUT.1
- new net N$3: Q5.1, R62.2, R63.2
- new net RX: J4.7, U3.36
- new net TX: J4.8, U3.37
- new net VIN: D16.C, D7.A, PWRIN.2, SWOUT.2
- net +24V: no longer VIN.1A, VIN.1B
- net 3V3: now also DEMP.3, J1.2, J4.2, J5.2, J6.2, LAT.3, R16.1, R24.1; no longer DE-EMPHASIS.3, I2CLCD.3, LATENCY.3, R16.2, R22.2
- net 5V: now also J1.4, J4.4, J5.4, J6.4
- net GND: now also DEMP.1, J1.1, J1.3, J4.1, J4.3, J5.1, J5.3, J6.1, J6.3, LAT.1, MODE.1, PWRIN.1, Q5.3, R63.1; no longer D7.A, DE-EMPHASIS.1, I2CLCD.4, IO0.1, LATENCY.1, VIN.2A, VIN.2B
- net IO0/BOOTMODE: now also MODE.3, R24.2; no longer IO0.3, R22.1
- net IO3/TWI_SDA: now also J6.9; no longer I2CLCD.2
- net IO4/TWI_SCK: now also J6.10; no longer I2CLCD.1
- net N$12: now also LAT.2; no longer LATENCY.2
- net N$13: now also DEMP.2; no longer DE-EMPHASIS.2
- net RESET: now also R16.2; no longer R16.1
Routing:
- net 5V: track 0.00 -> 131.3 mm
- net 3V3: track 197.5 -> 311.3 mm, vias 9 -> 8
- net IO3/TWI_SDA: track 0.00 -> 76.9 mm, vias 0 -> 1
- net IO46_PAUSE: track 0.00 -> 75.8 mm, vias 0 -> 1
- net IO9_STOP: track 0.00 -> 73.3 mm, vias 0 -> 1
- net IO4/TWI_SCK: track 0.00 -> 71.6 mm, vias 0 -> 2
- net IO8_PLAY: track 0.00 -> 70.6 mm, vias 0 -> 1
- net IO18_PREV: track 0.00 -> 68.6 mm, vias 0 -> 1
- net IO38_MOSFET: track 0.00 -> 67.6 mm, vias 0 -> 2
- net IO0/BOOTMODE: track 34.4 -> 99.9 mm, vias 0 -> 5
- net RESET: track 9.21 -> 65.1 mm, vias 0 -> 2
- net IO21_SHUFFLE: track 0.00 -> 53.2 mm, vias 0 -> 1
- net IO14_NEXT: track 0.00 -> 51.0 mm, vias 0 -> 1
- net IO16_LCD_D6: track 0.00 -> 49.6 mm, vias 0 -> 1
- net IO17_LCD_D7: track 0.00 -> 46.0 mm, vias 0 -> 1
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- added copper zone on layer 1, net +24V
- added copper zone on layer 1, net 5V-REG
- added copper zone on layer 1, net MOSFET-GND
- added copper zone on layer 1, net N$164
- added copper zone on layer 1, net VIN
Other:
- board size 100 x 100 mm -> 100 x 94.4 mm
- board text added: "(C) 2024"
- board text added: "-PWRIN+"
- board text added: "-SWOUT+"
- board text added: "1"
- board text added: "14"
- board text added: "15"
- board text added: "16"
- board text added: "17"
- board text added: "18"
- board text added: "2"
- board text added: "21"
- board text added: "3/SDA"
- board text added: "35"
- board text added: "36"
- board text added: "37"
- board text added: "3V3"
- board text added: "4/SCL"
- board text added: "45"
- board text added: "46"
- board text added: "47"
- board text added: "48"
- board text added: "5"
- board text added: "5V"
- board text added: "6"
- board text added: "7"
- board text added: "8"
- board text added: "9"
- board text added: "AUDIO DEVBOARD 1.0BETA MCU: ESP32S3 DAC: PCM5102A I2S MUTE: 39 I2S BCK: 40 I2S DATA: 41 I2S LRCK: 45 SD CS: 10 SD MOSI: 11 SD MISO: 12 SD SCK: 13 MOSFET: 38"
- board text added: "DIGITAL AUDIO CORE"
- board text added: "GND"
- board text added: "KAROO ELECTRONICS"
- board text added: "LINEOUT"
- board text added: "PORT A"
- board text added: "PORT B"
- board text added: "PORT C"
- board text added: "PORT D"
- board text added: "RX"
- board text added: "SDCARD"
- board text added: "TX"
- board text added: "USB"
- board text added: "V+"
- board text added: "V1.0BETA"

Commit message: sycned local
Other:
- board size 100 x 94.4 mm -> 100 x 98.4 mm
- board text added: "L"
- board text added: "R"
