File: I2S Audio Board/pcm5102_dac.sch (EAGLE design)
At the start: 61 parts, among them CON3 USB-C-Socket, IC1 PCM510xA, IC4 LM2596HV-5, IC5 AP2114H-3.3TRG1, J2 AUDIO_JACK_3.5MM_PTH, U3 ESP32S3WROOM1N8R8

Commit message: PCN5102 board
Parts:
- removed DE-EMPHASIS, LATENCY: (no value), SparkFun-Connectors2:CONN_03LOCK
- removed I2C, VIN: WJ212R-THR-3.5-2, WJ212R-THR-3.5-3.81:WJ212R-THR-3.5-2
- removed I2CLCD: MOLEX_SL_04-70555, molex-sl-connectors_jw:MOLEX_SL_04-70555
- removed R22: 10K, discrete:R-0603
- removed SPI: WJ212R-THR-3.5-3, WJ212R-THR-3.5-3.81:WJ212R-THR-3.5-3
- added CON7, CON8: PCB-2M3, Screw Terminals:PCB-2M3
- added D16: M4, diode:DIODE-DO-214AC
- added DEMP, LAT: (no value), jumper:SJ2W
- added J1, J4, J5, J6: (no value), SparkFun-Connectors:CONN_05X2SHD
- added PWRIN, SWOUT: Phoenix Pluggable 5.08mm 2 way, con-phoenix-508:MSTBA2
- added Q5: NCHAN, Cohesion_parts:N-POWER-MOSFETDPAK-MOSFET
- added R24: 10K, SparkFun-Resistors:5.1KOHM5.1KOHM-0603-1/10W-1%
- added R62: 10R, resistor:R-EU_R0603
- added R63: 100K, resistor:R-EU_R0603
- C42: value 10uF 50V -> 10uF
- R16: device discrete:R-0603 -> SparkFun-Resistors:5.1KOHM5.1KOHM-0603-1/10W-1%
- renumbered IO0 to MODE
Connections:
- new net IO1: J4.10, U3.IO1
- new net IO14_NEXT: J4.6, U3.IO14
- new net IO15_LCD_D5: J5.8, U3.IO15
- new net IO16_LCD_D6: J5.9, U3.IO16
- new net IO17_LCD_D7: J5.10, U3.IO17
- new net IO18_PREV: J6.5, U3.IO18
- new net IO2: J4.9, U3.IO2
- new net IO21_SHUFFLE: J4.5, U3.IO21
- new net IO35: J1.7, U3.IO35
- new net IO36: J1.6, U3.IO36
- new net IO37: J1.5, U3.IO37
- new net IO38_MOSFET: R62.1, U3.IO38
- new net IO45_LCD_BACKLIGHT: J1.8, U3.IO45
- new net IO46_PAUSE: J6.7, U3.IO46
- new net IO47_VOLM: J1.10, U3.IO47
- new net IO48_VOLP: J1.9, U3.IO48
- new net IO5_LCD_RS: J5.5, U3.IO5
- new net IO6_LCD_E: J5.6, U3.IO6
- new net IO7_LCD_D4: J5.7, U3.IO7
- new net IO8_PLAY: J6.6, U3.IO8
- new net IO9_STOP: J6.8, U3.IO9
- new net MOSFET-GND: D16.A, Q5.D, SWOUT-1.1
- new net N$3: Q5.G, R62.2, R63.2
- new net RX: J4.7, U3.RXD0
- new net TX: J4.8, U3.TXD0
- new net VIN: D16.C, D7.A, PWRIN-2.1, SWOUT-2.1
- net +24V: no longer VIN.P$1
- net 3V3: now also DEMP.3, J1.2, J4.2, J5.2, J6.2, LAT.3, R16.1, R24.1; no longer DE-EMPHASIS.3, I2CLCD.3, LATENCY.3, R16.2, R22.2
- net 5V: now also J1.4, J4.4, J5.4, J6.4
- net GND: now also DEMP.1, J1.1, J1.3, J4.1, J4.3, J5.1, J5.3, J6.1, J6.3, LAT.1, PWRIN-1.1, Q5.S, R63.1; no longer D7.A, DE-EMPHASIS.1, I2CLCD.4, LATENCY.1, VIN.P$2
- net IO0/BOOTMODE: now also R24.2; no longer R22.1
- net IO3/TWI_SDA: now also J6.9; no longer I2CLCD.2
- net IO4/TWI_SCK: now also J6.10; no longer I2CLCD.1
- net N$12: now also LAT.2; no longer LATENCY.2
- net N$13: now also DEMP.2; no longer DE-EMPHASIS.2
- net RESET: now also R16.2; no longer R16.1
Other:
- note added: "I2S DAC"
- note added: "MOSFET"
- note added: "MOUNTING"
- note added: "PWRIN"
- note added: "SD CARD"
- moved on the sheet: C1, C10, C11, C13, C15, C17, C2, C23, C24, C4, C42, C5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
